File: untitled.sch (EAGLE design)
At the start: 26 parts, among them J3 CORTEX_DEBUG_PTH, J6 USB-MICROB, U1 ATSAMD21G-M, U2 MIC5501-3.0YM5-TR, U3 TPD2S017, Y1 32.768KHZ

Commit message: Reselved VDDCORE error - rev 3
removed connection from vddcore to vcc that was causing a short burning out the internal arm regulator.
Connections:
- new net N$14: C1.1, U1.VDDCORE
- net VCC: no longer C1.1, U1.VDDCORE
Changed lines of the file:
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@@
 <part name="SUPPLY6" library="SparkFun-PowerSymbols" library_urn="urn:adsk.eagle:library:530" deviceset="VCC" device=""/>
 <part name="SUPPLY7" library="SparkFun-PowerSymbols" library_urn="urn:adsk.eagle:library:530" deviceset="VCC" device=""/>
-<part name="SUPPLY8" library="SparkFun-PowerSymbols" library_urn="urn:adsk.eagle:library:530" deviceset="VCC" device=""/>
 <part name="U2" library="MIC5501-3.0YM5-TR" deviceset="MIC5501-3.0YM5-TR" device=""/>
 <part name="R3" library="rcl" library_urn="urn:adsk.eagle:library:334" deviceset="R-US_" device="R0402" package3d_urn="urn:adsk.eagle:package:23547/2" value="10k"/>
@@
 <attribute name="VALUE" x="147.32" y="147.574" size="1.778" layer="96" align="bottom-center"/>
 </instance>
-<instance part="SUPPLY8" gate="G$1" x="154.94" y="142.24" smashed="yes">
-<attribute name="VALUE" x="154.94" y="145.034" size="1.778" layer="96" align="bottom-center"/>
-</instance>
 <instance part="U2" gate="G$1" x="116.84" y="200.66" smashed="yes">
 <attribute name="NAME" x="106.68" y="206.248" size="1.778" layer="95"/>
@@
 <junction x="147.32" y="144.78"/>
 <pinref part="SUPPLY7" gate="G$1" pin="VCC"/>
-</segment>
-<segment>
-<pinref part="U1" gate="G$1" pin="VDDCORE"/>
-<pinref part="C1" gate="G$1" pin="1"/>
-<wire x1="154.94" y1="142.24" x2="160.02" y2="142.24" width="0.1524" layer="91"/>
-<junction x="154.94" y="142.24"/>
-<junction x="160.02" y="142.24"/>
-<pinref part="SUPPLY8" gate="G$1" pin="VCC"/>
 </segment>
 <segment>
@@
 </segment>
 </net>
+<net name="N$14" class="0">
+<segment>
+<pinref part="U1" gate="G$1" pin="VDDCORE"/>
+<pinref part="C1" gate="G$1" pin="1"/>
+<wire x1="154.94" y1="142.24" x2="160.02" y2="142.24" width="0.1524" layer="91"/>
+<junction x="160.02" y="142.24"/>
+<junction x="154.94" y="142.24"/>
+</segment>
+</net>
