File: devils-rectangle.brd (EAGLE design)
At the start: 54 x 54 mm, 27 parts, among them IC1 74AHC1G125DBV, J3 CORTEX_DEBUG_PTH, J6 USB-MICROB, U1 ATSAMD21G-M, U2 MIC5501-3.0YM5-TR, U3 TPD2S017, Y1 32.768KHZ

Commit message: rev 3
fixed errors, sent to fab.
Parts:
- removed C4, C5: 7pf, SparkFun-Capacitors:0402
- removed Y1: 32.768KHZ, Seeed-Crystal Oscillator:X2-SMD-3.2X1.5X0.55MM
Connections:
- removed net N$12: C5.2, U1.2, Y1.1
- removed net N$13: C4.2, U1.1, Y1.2
- removed net PA08: J5.3
- new net PA03: J5.3, U1.4
- net GND: no longer C4.1, C5.1
Routing:
- net PA03: track 0.00 -> 9.29 mm, vias 0 -> 1
- net N$12: track 5.28 -> 0.00 mm
- net N$13: track 5.26 -> 0.00 mm
- net GND: track 62.3 -> 61.4 mm
Changed lines of the file:
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@@
 <attribute name="VALUE" x="10.165" y="26.955" size="0.6096" layer="28" rot="MR180"/>
-</element>
-<element name="Y1" library="Seeed-Crystal Oscillator" library_urn="urn:adsk.eagle:library:466" package="X2-SMD-3.2X1.5X0.55MM" package3d_urn="urn:adsk.eagle:package:32493/1" value="32.768KHZ" x="33" y="11.5" smashed="yes" rot="MR90">
-<attribute name="MPN" value="FC-135" x="33" y="11.5" size="0.8128" layer="28" rot="MR90" display="off"/>
-<attribute name="NAME" x="31.516" y="10.849" size="0.6096" layer="26" ratio="11" rot="MR90"/>
-</element>
-<element name="C4" library="SparkFun-Capacitors" library_urn="urn:adsk.eagle:library:510" package="0402" package3d_urn="urn:adsk.eagle:package:37413/1" value="7pf" x="35.5" y="12.5" smashed="yes" rot="MR0">
-<attribute name="NAME" x="35.5" y="13.262" size="0.6096" layer="26" font="vector" ratio="20" rot="MR0" align="bottom-center"/>
-<attribute name="PROD_ID" value="CAP-12416" x="35.5" y="12.5" size="0.8128" layer="28" rot="MR0" display="off"/>
-<attribute name="VALUE" x="36.762" y="12.5" size="0.6096" layer="28" font="vector" ratio="20" rot="MR270" align="top-center"/>
-</element>
-<element name="C5" library="SparkFun-Capacitors" library_urn="urn:adsk.eagle:library:510" package="0402" package3d_urn="urn:adsk.eagle:package:37413/1" value="7pf" x="35.5" y="10.5" smashed="yes" rot="MR0">
-<attribute name="NAME" x="35.5" y="11.262" size="0.6096" layer="26" font="vector" ratio="20" rot="MR0" align="bottom-center"/>
-<attribute name="PROD_ID" value="CAP-12416" x="35.5" y="10.5" size="0.8128" layer="28" rot="MR0" display="off"/>
-<attribute name="VALUE" x="36.762" y="10.5" size="0.6096" layer="28" font="vector" ratio="20" rot="MR270" align="top-center"/>
 </element>
 <element name="IC1" library="74xx-custom" package="SOT23-5" package3d_urn="urn:adsk.eagle:package:2482/1" value="74AHC1G125DBV" x="24.5" y="3.5" smashed="yes" rot="R90">
@@
 <wire x1="22.1" y1="10.6" x2="21" y2="9.5" width="0.254" layer="1"/>
 <via x="21" y="9.5" extent="1-16" drill="0.35"/>
-<contactref element="C5" pad="1"/>
-<contactref element="C4" pad="1"/>
 <wire x1="30.4" y1="9.75" x2="31.55" y2="9.75" width="0.254" layer="16"/>
 <wire x1="31.55" y1="9.75" x2="32.25" y2="9.05" width="0.254" layer="16"/>
@@
 <wire x1="33.75" y1="9.05" x2="34" y2="9.3" width="0.254" layer="16"/>
 <wire x1="34" y1="9.3" x2="35.8" y2="9.3" width="0.254" layer="16"/>
-<wire x1="36.08" y1="9.58" x2="36.08" y2="10.5" width="0.254" layer="16"/>
 <wire x1="35.8" y1="9.3" x2="36.08" y2="9.58" width="0.254" layer="16"/>
 <contactref element="IC1" pad="3"/>
@@
 <contactref element="J3" pad="10"/>
 <wire x1="23.925" y1="15.075" x2="20.075" y2="15.075" width="0.254" layer="16"/>
-<wire x1="25.75" y1="12.4" x2="25.7544" y2="12.4044" width="0.254" layer="16"/>
 <via x="25.2" y="15.2" extent="1-16" drill="0.35"/>
 <wire x1="35.54" y1="15.365" x2="35.54" y2="15.02144375" width="0.254" layer="1"/>
@@
 <wire x1="13.52" y1="6.58" x2="13.5" y2="6.58" width="0.3048" layer="16"/>
 </signal>
-<signal name="PA08">
-<contactref element="J5" pad="3"/>
-<wire x1="39.47" y1="9.97" x2="39.53" y2="9.97" width="0.254" layer="16"/>
-</signal>
 <signal name="PA09">
 <contactref element="U1" pad="8"/>
@@
 <wire x1="12" y1="28" x2="12" y2="37.61" width="0.254" layer="1"/>
 <wire x1="12" y1="37.61" x2="11.76" y2="37.85" width="0.254" layer="1"/>
-</signal>
-<signal name="N$12">
-<contactref element="U1" pad="2"/>
-<contactref element="Y1" pad="1"/>
-<contactref element="C5" pad="2"/>
-<wire x1="33" y1="10" x2="33" y2="9.976" width="0.254" layer="16"/>
-<wire x1="33" y1="9.976" x2="34.396" y2="9.976" width="0.254" layer="16"/>
-<wire x1="34.396" y1="9.976" x2="34.92" y2="10.5" width="0.254" layer="16"/>
-<wire x1="30.4" y1="11.25" x2="31.28881875" y2="11.25" width="0.254" layer="16"/>
-<wire x1="32.53881875" y1="10" x2="33" y2="10" width="0.254" layer="16"/>
-<wire x1="31.28881875" y1="11.25" x2="32.53881875" y2="10" width="0.254" layer="16"/>
-</signal>
-<signal name="N$13">
-<contactref element="U1" pad="1"/>
-<contactref element="Y1" pad="2"/>
-<contactref element="C4" pad="2"/>
-<wire x1="30.4" y1="11.75" x2="31.3" y2="11.75" width="0.254" layer="16"/>
-<wire x1="32.574" y1="13.024" x2="33" y2="13.024" width="0.254" layer="16"/>
-<wire x1="31.3" y1="11.75" x2="32.574" y2="13.024" width="0.254" layer="16"/>
-<wire x1="34.92" y1="12.5" x2="34.396" y2="13.024" width="0.254" layer="16"/>
-<wire x1="34.396" y1="13.024" x2="33" y2="13.024" width="0.254" layer="16"/>
 </signal>
 <signal name="N$14">
@@
 <wire x1="23" y1="8.5" x2="23" y2="7.85" width="0.254" layer="1"/>
 </signal>
+<signal name="PA03">
+<contactref element="U1" pad="4"/>
+<contactref element="J5" pad="3"/>
+<wire x1="30.4" y1="10.25" x2="33.55" y2="10.25" width="0.254" layer="16"/>
+<wire x1="33.55" y1="10.25" x2="33.85" y2="9.95" width="0.254" layer="16"/>
+<wire x1="33.85" y1="9.95" x2="33.9" y2="10" width="0.254" layer="16"/>
+<wire x1="33.9" y1="10" x2="34" y2="10" width="0.254" layer="16"/>
+<via x="34" y="10" extent="1-16" drill="0.35"/>
+<wire x1="34" y1="10" x2="39.5" y2="10" width="0.254" layer="1"/>
+<wire x1="39.5" y1="10" x2="39.53" y2="9.97" width="0.254" layer="1"/>
+</signal>
 </signals>
